Commit message: urdf modify

File: spot_micro_description/urdf/spotmicroai_gen_ros.urdf (robot description, URDF)
Before this commit: robot SpotMicroAI, 25 links, 24 joints
Links:
- link rear_right_leg_link_cover: geometry collision box size=0.028 0.036 0.12; collision mesh filename=package://spot_micro_description/urdf/stl/rarm_cover.stl scale=0.001 0.001 0.001

Commit message: modify

File: spot_micro_description/urdf/spotmicroai_gen_ros.urdf (robot description, URDF)
Before this commit: robot SpotMicroAI, 25 links, 24 joints
Joints:
- joint rear_right_leg_cover_joint: origin xyz=0 0 0 -> xyz=0 0 0 rpy=0 0 0
